File: linky_wb.kicad_pcb (KiCad board)
At the start: 4 copper layers, 24 x 40 mm, 66 parts, among them J1 Conn_01x03_Pin, J2 Conn_02x05_Counter_Clockwise, Q1 BS170F, SW1 SW1, U1 TPS78230DDC, U2 MCP9700AT-ETT, U3 STM32WB55RGVx, Y1 nx2012_32768, Y2 nx2016_32m

Commit message: erc/drc: fixes & regen
Parts:
- removed kibuzzard-670D0979: G***, kibuzzard-670D0979
- removed kibuzzard-670D11FE: G***, kibuzzard-670D11FE
- added kibuzzard-670D18C1: G***, kibuzzard-670D18C1, F.Cu at (173.2, 55.9)
- added kibuzzard-670D18F3: G***, kibuzzard-670D18F3, F.Cu at (173.2, 53.8)
- moved L3 0.61 mm to (172.1, 83.5)
- moved L2 0.52 mm to (170.7, 83.9)
- moved L1 0.40 mm to (169.3, 83.5)
- moved AE3 0.31 mm to (169.2, 84.8)
Routing:
- net GND: track 44.2 -> 45.3 mm, vias 63 -> 62

Commit message: 1.0.0 boards sent to production
Parts:
- C17: value 10uF 6.3v -> 4.7uF
- R1, R13: value 5.1k -> 10k
- R10: value 330 -> 0
- R12, R5, R6, R9: value 5.1k -> 1.5k
- R7: value 220k -> 10k
- moved kibuzzard-670D18C1 67.0 mm to (110.0, 33.8)
- moved kibuzzard-670D18F3 67.0 mm to (110.0, 31.8)
- moved kibuzzard-670CFC68 66.8 mm to (100.8, 41.2)
- moved kibuzzard-670CFC05 66.8 mm to (98.2, 41.2)
- moved kibuzzard-670CFC0C 66.8 mm to (95.7, 41.2)
- moved kibuzzard-670CFCA8 66.8 mm to (105.4, 39.2)
- moved L3 66.8 mm to (109.1, 61.4)
- moved L2 66.8 mm to (107.7, 61.9)
- moved C1 66.7 mm to (113.3, 47.3)
- moved C13 66.7 mm to (104.4, 55.7)
- moved C5 66.7 mm to (99.7, 43.5)
- moved C7 66.7 mm to (102.9, 51.4)
- moved C9 66.7 mm to (105.1, 49.1)
- moved D2 66.7 mm to (108.3, 44.0)
- moved D6 66.7 mm to (100.8, 54.7)
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Connections:
- net Net-(AE2-OUT) renamed /wb55/ant_path
- net Net-(AE3-A) renamed /wb55/pi_to_ant
- net Net-(J1-Pin_1) renamed /I1
- net Net-(J1-Pin_2) renamed /I2
- net Net-(J1-Pin_3) renamed /A
- AE3 pad 2: GND -> (no net)
- J2 pad 5: +5V -> unconnected-(J2-Pin_5-Pad5)
Routing:
- net GND: track 45.3 -> 42.9 mm, vias 62 -> 75
- net VDD: track 49.2 -> 49.8 mm
Other:
- outline, holes or cut-outs redrawn

Commit message: cleanups, exclude some drcs, fix antenna symbol to avoid ground disconnection, tweak ci
Parts:
- L1, L3: value L -> tbd
- L2: value L -> 0
- Y1: value nx2012_32768 -> nx2012 32.768khz
- Y2: value nx2016_32m -> NX2016SA 32.0Mhz EXS00A-CS06465
Connections:
- AE3 pad 2: (no net) -> GND
- D2 pad 3: /A -> GND
- J1 pad 3: /A -> GND
Routing:
- net GND: track 42.9 -> 60.0 mm, vias 75 -> 76
- net /A: track 17.2 -> 0.00 mm, vias 1 -> 0
